Commit message: Added the kinect meshes.

File: au_automow_common/automow_description/urdf/lawnmower.xacro (robot description, xacro)
@@ -1,4 +1,5 @@
 <?xml version="1.0"?>
-<robot>
+<robot
+    xmlns:xacro="http://playerstage.sourceforge.net/gazebo/xmlschema/#interface" name="macroed">
     <material name="Green">
         <color rgba="0.0 0.8 0.0 1.0"/>
@@ -14,147 +15,117 @@
     </material>
     <property name="M_PI" value="3.14159"/>
-    <macro name="automow">
-        <!-- base_footprint is a ficticious frame on the ground below base_link
-             for the navigation stack to properly function -->
-        <link name="base_footprint">
-            <inertial>
-                <mass value="0.0001" />
-                <origin xyz="0 0 0" />
-                <inertia ixx="0.0001" ixy="0.0" ixz="0.0"
-                         iyy="0.0001" iyz="0.0"
-                         izz="0.0001" />
-             </inertial>
-             <visual>
-                 <origin xyz="0 0 0" rpy="0 0 0" />
-                 <geometry>
-                     <box size="0.001 0.001 0.001" />
-                 </geometry>
-                 <material name="Green" />
-             </visual>
-             <collision>
-                  <origin xyz="0 0 0" rpy="0 0 0" />
-                 <geometry>
-                     <box size="0.001 0.001 0.001" />
-                 </geometry>
-             </collision>
-         </link>
-         <!-- base_link is the origin for all of the coordinates on the robot.
-              For our case, this will be centered under the wheels of the
-              robot. -->
-         <link name="base_link">
-             <inertial>
-                 <mass value="100" />
-                 <origin xyz="0 0 0.063" />
-                 <inertia ixx="1.0" ixy="0.0" ixz="0.0"
-                          iyy="1.0" iyz="0.0"
-                          izz="1.0" />
-              </inertial>
-              <visual>
-                  <origin xyz="0 0 0.0308" rpy="0 0 0" />
-              </visual>
-          </link>
-          <link name="left_wheel_link"/>
-          <link name="right_wheel_link"/>
-          <link name="laser" />
-          <link name="ahrs" />
-          <joint name="base_footprint_joint" type="fixed">
-              <parent link="base_footprint"/>
-              <child link="base_link"/>
-          </joint>
-          <joint name="left_wheel_joint" type="continuous">
-              <parent link="base_link"/>
-              <child link="left_wheel_link"/>
-          </joint>
-          <joint name="right_wheel_joint" type="continuous">
-              <parent link="base_link"/>
-              <child link="right_wheel_link"/>
-          </joint>
-          <joint name="laser_joint" type="fixed">
-              <parent link="base_link" />
-              <child link="laser" />
-          </joint>
-          <joint name="ahrs_joint" type="fixed">
-              <parent link="base_link" />
-              <child link="ahrs" />
-          </joint>
-          <link name="kinect_link">
-              <inertial>
-                  <mass value="0.00001" />
-                  <origin xyz="0 0 0" />
-                  <inertia ixx="1.0" ixy="0.0" ixz="0.0"
-                          iyy="1.0" iyz="0.0"
-                          izz="1.0" />
-              </inertial>
-              <visual>
-                  <origin xyz="0 0 0" rpy="0 0 0"/>
-                  <geometry>
-                      <mesh
-                          filename="package://automow_description/meshes/kinect.dae"/>
-                  </geometry>
-              </visual>
-              <collision>
-                  <origin xyz="0 0 0" rpy="0 0 0"/>
-                  <geometry>
-                      <box size="0.0730 0.2760 0.0720"/>
-                  </geometry>
-              </collision>
-          </link>
-          <link name="kinect_depth_frame">
-              <inertial>
-                  <mass value="0.000001" />
-                  <origin xyz="0 0 0" />
-                  <inertia ixx="1.0" ixy="0.0" ixz="0.0"
-                          iyy="1.0" iyz="0.0"
-                          izz="1.0" />
-              </inertial>
-          </link>
-          <link name="kinect_depth_optical_frame">
-              <inertial>
-                  <mass value="0.000001" />
-                  <origin xyz="0 0 0" />
-                  <inertia ixx="1.0" ixy="0.0" ixz="0.0"
-                          iyy="1.0" iyz="0.0"
-                          izz="1.0" />
-              </inertial>
-          </link>
-          <link name="kinect_rgb_frame">
-              <inertial>
-                  <mass value="0.000001" />
-                  <origin xyz="0 0 0" />
-                  <inertia ixx="1.0" ixy="0.0" ixz="0.0"
-                          iyy="1.0" iyz="0.0"
-                          izz="1.0" />
-              </inertial>
-          </link>
-          <link name="kinect_rgb_optical_frame">
-               <inertial>
-                  <mass value="0.000001" />
-                  <origin xyz="0 0 0" />
-                  <inertia ixx="1.0" ixy="0.0" ixz="0.0"
-                          iyy="1.0" iyz="0.0"
-                          izz="1.0" />
-              </inertial>
-          </link>
-          <joint name="base_kinect_joint" type="fixed">
-          </joint>
-          <joint name="kinect_depth_joint" type="fixed">
-              <parent link="kinect_link" />
-              <child link="kinect_depth_frame" />
-          </joint>
-          <joint name="kinect_depth_optical_joint" type="fixed">
-              <origin xyz="0 0 0" rpy="${-M_PI/2} 0 ${M_PI/2}"/>
-              <parent link="kinect_depth_frame" />
-              <child link="kinect_depth_optical_frame" />
-          </joint>
-          <joint name="kinect_rgb_joint" type="fixed">
-              <origin xyz="0 -0.005 0" rpy="0 0 0" />
-              <parent link="kinect_link" />
-              <child link="kinect_rgb_frame" />
-          </joint>
-          <joint name="kinect_rgb_optical_joint" type="fixed">
-              <origin xyz="0 0 0" rpy="${-M_PI/2} 0 ${M_PI/2}"/>
-              <parent link="kinect_rgb_frame" />
-              <child link="kinect_rgb_optical_frame" />
-          </joint>
-      </macro>
-  </robot>
+    <xacro:macro name="default_inertial" params="mass">
+        <inertial>
+            <mass value="${mass}" />
+            <inertia ixx="1.0" ixy="0.0" ixz="0.0"
+                     iyy="1.0" iyz="0.0"
+                     izz="1.0" />
+        </inertial>
+    </xacro:macro>
+    <!-- base_footprint is a ficticious frame on the ground below base_link
+     for the navigation stack to properly function -->
+    <link name="base_footprint">
+        <inertial>
+        <mass value="0.0001" />
+        <origin xyz="0 0 0" />
+        <inertia ixx="0.0001" ixy="0.0" ixz="0.0"
+                 iyy="0.0001" iyz="0.0"
+                 izz="0.0001" />
+        </inertial>
+        <visual>
+         <origin xyz="0 0 0" rpy="0 0 0" />
+         <geometry>
+             <box size="0.001 0.001 0.001" />
+         </geometry>
+         <material name="Green" />
+        </visual>
+        <collision>
+          <origin xyz="0 0 0" rpy="0 0 0" />
+         <geometry>
+             <box size="0.001 0.001 0.001" />
+         </geometry>
+        </collision>
+    </link>
+    <!-- base_link is the origin for all of the coordinates on the robot.
+      For our case, this will be centered under the wheels of the
+      robot. -->
+    <link name="base_link">
+        <xacro:default_inertial mass="100"/>
+        <visual>
+            <origin xyz="0 0 0.0308" rpy="0 0 0" />
+        </visual>
+    </link>
+    <link name="left_wheel_link"/>
+    <link name="right_wheel_link"/>
+    <link name="laser" />
+    <link name="ahrs" />
+    <joint name="base_footprint_joint" type="fixed">
+        <parent link="base_footprint"/>
+        <child link="base_link"/>
+    </joint>
+    <joint name="left_wheel_joint" type="continuous">
+        <parent link="base_link"/>
+        <child link="left_wheel_link"/>
+    </joint>
+    <joint name="right_wheel_joint" type="continuous">
+        <parent link="base_link"/>
+        <child link="right_wheel_link"/>
+    </joint>
+    <joint name="laser_joint" type="fixed">
+        <parent link="base_link" />
+        <child link="laser" />
+    </joint>
+    <joint name="ahrs_joint" type="fixed">
+        <parent link="base_link" />
+        <child link="ahrs" />
+    </joint>
+    <link name="kinect_link">
+        <xacro:default_inertial mass="0.0001"/>
+        <visual>
+            <origin xyz="0 0 0" rpy="0 0 0"/>
+            <geometry>
+                <mesh
+                  filename="package://automow_description/meshes/kinect.dae"/>
+            </geometry>
+        </visual>
+        <collision>
+            <origin xyz="0 0 0" rpy="0 0 0"/>
+            <geometry>
+                <box size="0.0730 0.2760 0.0720"/>
+            </geometry>
+        </collision>
+    </link>
+    <link name="kinect_depth_frame">
+        <xacro:default_inertial mass="0.000001"/>
+    </link>
+    <link name="kinect_depth_optical_frame">
+        <xacro:default_inertial mass="0.000001"/>
+    </link>
+    <link name="kinect_rgb_frame">
+        <xacro:default_inertial mass="0.000001"/>
+    </link>
+    <link name="kinect_rgb_optical_frame">
+        <xacro:default_inertial mass="0.000001"/>
+    </link>
+    <joint name="base_kinect_joint" type="fixed">
+    </joint>
+    <joint name="kinect_depth_joint" type="fixed">
+      <parent link="kinect_link" />
+      <child link="kinect_depth_frame" />
+    </joint>
+    <joint name="kinect_depth_optical_joint" type="fixed">
+      <origin xyz="0 0 0" rpy="${-M_PI/2} 0 ${M_PI/2}"/>
+      <parent link="kinect_depth_frame" />
+      <child link="kinect_depth_optical_frame" />
+    </joint>
+    <joint name="kinect_rgb_joint" type="fixed">
+      <origin xyz="0 -0.005 0" rpy="0 0 0" />
+      <parent link="kinect_link" />
+      <child link="kinect_rgb_frame" />
+    </joint>
+    <joint name="kinect_rgb_optical_joint" type="fixed">
+      <origin xyz="0 0 0" rpy="${-M_PI/2} 0 ${M_PI/2}"/>
+      <parent link="kinect_rgb_frame" />
+      <child link="kinect_rgb_optical_frame" />
+    </joint>
+</robot>

Commit message: Working xacro file, at least.

File: au_automow_common/automow_description/urdf/lawnmower.xacro (robot description, xacro)
@@ -1,5 +1,6 @@
 <?xml version="1.0"?>
 <robot
-    xmlns:xacro="http://playerstage.sourceforge.net/gazebo/xmlschema/#interface" name="macroed">
+    xmlns:xacro="http://playerstage.sourceforge.net/gazebo/xmlschema/#interface"
+    name="automow">
     <material name="Green">
         <color rgba="0.0 0.8 0.0 1.0"/>
@@ -14,5 +15,11 @@
         <color rgba="0.0 0.0 0.8 1.0"/>
     </material>
-    <property name="M_PI" value="3.14159"/>
+    <material name="Black">
+        <color rgba="0.0 0.0 0.0 1.0"/>
+    </material>
+    <material name="Grey">
+        <color rgba="0.7 0.7 0.7 0.7"/>
+    </material>
+    <xacro:property name="M_PI" value="3.14159"/>
     <xacro:macro name="default_inertial" params="mass">
         <inertial>
@@ -50,31 +57,90 @@
       For our case, this will be centered under the wheels of the
       robot. -->
+    <xacro:property name="clearance" value="0.065" />
+    <xacro:property name="c_width" value="0.51" />
+    <xacro:property name="c_length" value="0.73" />
+    <xacro:property name="c_height" value="0.54" />
     <link name="base_link">
         <xacro:default_inertial mass="100"/>
         <visual>
-            <origin xyz="0 0 0.0308" rpy="0 0 0" />
-        </visual>
-    </link>
-    <link name="left_wheel_link"/>
-    <link name="right_wheel_link"/>
-    <link name="laser" />
-    <link name="ahrs" />
+            <origin xyz="${c_length/2} ${c_width/2} ${c_height/2}" rpy="0 0 0" />
+            <geometry>
+                <box size="${c_length} ${c_width} ${c_height}" />
+            </geometry>
+            <material name="Grey" />
+        </visual>
+        <collision>
+            <origin xyz="${c_length/2} ${c_width/2} ${c_height/2}" rpy="0 0 0" />
+            <geometry>
+                <box size="${c_length} ${c_width} ${c_height}" />
+            </geometry>
+        </collision>
+    </link>
     <joint name="base_footprint_joint" type="fixed">
+        <origin xyz="0 0 ${clearance}" rpy="0 0 0"/>
         <parent link="base_footprint"/>
         <child link="base_link"/>
     </joint>
-    <joint name="left_wheel_joint" type="continuous">
-        <parent link="base_link"/>
-        <child link="left_wheel_link"/>
-    </joint>
-    <joint name="right_wheel_joint" type="continuous">
-        <parent link="base_link"/>
-        <child link="right_wheel_link"/>
-    </joint>
+    <xacro:property name="wheeldiam" value="30"/>
+    <xacro:macro name="wheel" params="prefix reflect">
+        <link name="${prefix}_wheel_link">
+            <visual>
+                <geometry>
+                    <cylinder radius="${wheeldiam/2}" length="0.1"/>
+                </geometry>
+                <material name="Black"/>
+            </visual>
+            <collision>
+                <geometry>
+                    <cylinder radius="${wheeldiam/2}" length="0.1"/>
+                </geometry>
+            </collision>
+            <xacro:default_inertial mass="1"/>
+        </link>
+        <joint name="${prefix}_wheel_joint">
+            <axis xyz="0 0 1"/>
+            <parent link="base_link"/>
+            <child link="${prefix}_wheel_link"/>
+            <origin xyz="0 ${c_width*reflect/2 + 1} ${wheeldiam/2 + clearance}"
+                rpy="0 0 0"/>
+        </joint>
+    </xacro:macro>
+    <link name="laser">
+        <visual>
+            <origin xyz="0 0 -0.07" />
+            <geometry>
+                <cylinder radius="0.06" length="0.08"/>
+            </geometry>
+            <material name="Red"/>
+        </visual>
+        <collision>
+            <origin xyz="0 0 -0.07" />
+            <geometry>
+                <cylinder radius="0.06" length="0.08"/>
+            </geometry>
+        </collision>
+        <xacro:default_inertial mass="0.5"/>
+    </link>
+    <link name="ahrs">
+        <visual>
+            <geometry>
+                <box size="0.02 0.02 0.02"/>
+            </geometry>
+            <material name="Black"/>
+        </visual>
+        <collision>
+            <geometry>
+                <box size="0.02 0.02 0.02"/>
+            </geometry>
+        </collision>
+        <xacro:default_inertial mass="0.001"/>
+    </link>
     <joint name="laser_joint" type="fixed">
+        <origin xyz="81.5 0 21.5" rpy="0 0 0"/>
         <parent link="base_link" />
         <child link="laser" />
     </joint>
     <joint name="ahrs_joint" type="fixed">
+        <origin xyz="22 0 ${c_height - 2}" rpy="${M_PI/2} 0 0"/>
         <parent link="base_link" />
         <child link="ahrs" />
@@ -109,13 +175,17 @@
     </link>
     <joint name="base_kinect_joint" type="fixed">
+        <origin xyz="0.49  0.005 ${c_height + 0.05}" rpy="0 ${M_PI/12} 0"/>
+        <parent link="base_link"/>
+        <child link="kinect_link"/>
     </joint>
     <joint name="kinect_depth_joint" type="fixed">
-      <parent link="kinect_link" />
-      <child link="kinect_depth_frame" />
+        <origin xyz="0 0.018 0" rpy="0 0 0" />
+        <parent link="kinect_link" />
+        <child link="kinect_depth_frame" />
     </joint>
     <joint name="kinect_depth_optical_joint" type="fixed">
-      <origin xyz="0 0 0" rpy="${-M_PI/2} 0 ${M_PI/2}"/>
-      <parent link="kinect_depth_frame" />
-      <child link="kinect_depth_optical_frame" />
+        <origin xyz="0 0 0" rpy="${-M_PI/2} 0 ${M_PI/2}"/>
+        <parent link="kinect_depth_frame" />
+        <child link="kinect_depth_optical_frame" />
     </joint>
     <joint name="kinect_rgb_joint" type="fixed">
